File: hw/eagle/projects/size_M/ext_rgb/ext_rgb_M.brd (EAGLE design)
At the start: 30 x 30 mm, 6 parts

Commit message: completed pcb design for M.0 - made PCB order
Parts:
- removed JP1: (no value), pinhead2:1X04
- added JP3: (no value), pinhead2:1X05
- R1, R2, R3: value (none) -> 330
- moved R3 0.41 mm to (5.31, 12.1)
- moved R1 0.33 mm to (5.33, 16.5)
- moved JP2 0.10 mm to (1.40, 13.0)
Connections:
- new net VDD: JP3.4
- net GND: now also JP2.6, JP3.3; no longer JP1.2
Routing:
- net GND: track 12.1 -> 33.5 mm
Other:
- board outline removed
