File: hw/eagle/projects/size_M/ext_rgb/ext_rgb_M.sch (EAGLE design)
At the start: 6 parts

Commit message: completed pcb design for M.0 - made PCB order
Parts:
- removed JP1: (no value), pinhead2:PINHD-1X4
- added JP3: (no value), pinhead2:PINHD-1X5
- R1, R2, R3: value (none) -> 330
Connections:
- new net VDD: JP3.4
- net GND: now also JP2.6, JP3.3; no longer JP1.2
Other:
- moved on the sheet: JP2, R1, R2
Changed lines of the file:
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@@
 </classes>
 <parts>
-<part name="JP1" library="pinhead2" deviceset="PINHD-1X4" device="" package3d_urn="urn:adsk.eagle:package:22407/2"/>
 <part name="JP2" library="pinhead2" deviceset="PINHD-1X6" device="" package3d_urn="urn:adsk.eagle:package:22472/2"/>
 <part name="U$2" library="!stavebnice03" deviceset="RGB_WW-FCE50TC-Q1" device=""/>
-<part name="R1" library="resistor" deviceset="R-EU_" device="R0603"/>
-<part name="R2" library="resistor" deviceset="R-EU_" device="R0603"/>
-<part name="R3" library="resistor" deviceset="R-EU_" device="R0603"/>
+<part name="R1" library="resistor" deviceset="R-EU_" device="R0603" value="330"/>
+<part name="R2" library="resistor" deviceset="R-EU_" device="R0603" value="330"/>
+<part name="R3" library="resistor" deviceset="R-EU_" device="R0603" value="330"/>
+<part name="JP3" library="pinhead2" deviceset="PINHD-1X5" device="" package3d_urn="urn:adsk.eagle:package:22469/2"/>
 </parts>
 <sheets>
@@
 </plain>
 <instances>
-<instance part="JP1" gate="A" x="48.26" y="43.18" smashed="yes">
-<attribute name="NAME" x="41.91" y="51.435" size="1.778" layer="95"/>
-<attribute name="VALUE" x="41.91" y="35.56" size="1.778" layer="96"/>
-</instance>
-<instance part="JP2" gate="A" x="-17.78" y="48.26" smashed="yes" rot="R180">
-<attribute name="NAME" x="-11.43" y="37.465" size="1.778" layer="95" rot="R180"/>
-<attribute name="VALUE" x="-11.43" y="58.42" size="1.778" layer="96" rot="R180"/>
+<instance part="JP2" gate="A" x="-15.24" y="48.26" smashed="yes" rot="R180">
+<attribute name="NAME" x="-8.89" y="37.465" size="1.778" layer="95" rot="R180"/>
+<attribute name="VALUE" x="-8.89" y="58.42" size="1.778" layer="96" rot="R180"/>
 </instance>
 <instance part="U$2" gate="G$1" x="17.78" y="60.96" smashed="yes" rot="R180">
 <attribute name="NAME" x="27.94" y="66.04" size="1.27" layer="94" rot="R270"/>
 </instance>
-<instance part="R1" gate="G$1" x="5.08" y="81.28" smashed="yes" rot="MR180">
-<attribute name="NAME" x="1.27" y="79.7814" size="1.778" layer="95" rot="MR180"/>
-<attribute name="VALUE" x="1.27" y="84.582" size="1.778" layer="96" rot="MR180"/>
+<instance part="R1" gate="G$1" x="5.08" y="86.36" smashed="yes" rot="MR180">
+<attribute name="NAME" x="1.27" y="84.8614" size="1.778" layer="95" rot="MR180"/>
+<attribute name="VALUE" x="1.27" y="89.662" size="1.778" layer="96" rot="MR180"/>
 </instance>
-<instance part="R2" gate="G$1" x="5.08" y="76.2" smashed="yes" rot="MR180">
-<attribute name="NAME" x="1.27" y="74.7014" size="1.778" layer="95" rot="MR180"/>
-<attribute name="VALUE" x="1.27" y="79.502" size="1.778" layer="96" rot="MR180"/>
+<instance part="R2" gate="G$1" x="5.08" y="78.74" smashed="yes" rot="MR180">
+<attribute name="NAME" x="1.27" y="77.2414" size="1.778" layer="95" rot="MR180"/>
+<attribute name="VALUE" x="1.27" y="82.042" size="1.778" layer="96" rot="MR180"/>
 </instance>
 <instance part="R3" gate="G$1" x="5.08" y="71.12" smashed="yes" rot="MR180">
 <attribute name="NAME" x="1.27" y="69.6214" size="1.778" layer="95" rot="MR180"/>
 <attribute name="VALUE" x="1.27" y="74.422" size="1.778" layer="96" rot="MR180"/>
+</instance>
+<instance part="JP3" gate="A" x="38.1" y="45.72" smashed="yes">
+<attribute name="NAME" x="31.75" y="53.975" size="1.778" layer="95"/>
+<attribute name="VALUE" x="31.75" y="35.56" size="1.778" layer="96"/>
 </instance>
 </instances>
@@
 <net name="N$3" class="0">
 <segment>
-<wire x1="17.78" y1="76.2" x2="10.16" y2="76.2" width="0.1524" layer="91"/>
+<wire x1="17.78" y1="78.74" x2="10.16" y2="78.74" width="0.1524" layer="91"/>
 <pinref part="R2" gate="G$1" pin="2"/>
 <pinref part="U$2" gate="G$1" pin="2"/>
-<wire x1="17.78" y1="76.2" x2="17.78" y2="71.12" width="0.1524" layer="91"/>
+<wire x1="17.78" y1="78.74" x2="17.78" y2="71.12" width="0.1524" layer="91"/>
 </segment>
 </net>
@@
 <wire x1="22.86" y1="48.26" x2="22.86" y2="45.72" width="0.1524" layer="91"/>
 <junction x="22.86" y="45.72"/>
-<pinref part="JP1" gate="A" pin="2"/>
-<wire x1="45.72" y1="45.72" x2="22.86" y2="45.72" width="0.1524" layer="91"/>
+<wire x1="35.56" y1="45.72" x2="22.86" y2="45.72" width="0.1524" layer="91"/>
 <junction x="22.86" y="45.72"/>
+<pinref part="JP3" gate="A" pin="3"/>
+<pinref part="JP2" gate="A" pin="6"/>
+<wire x1="-12.7" y1="53.34" x2="7.62" y2="53.34" width="0.1524" layer="91"/>
+<wire x1="7.62" y1="53.34" x2="7.62" y2="45.72" width="0.1524" layer="91"/>
+<wire x1="7.62" y1="45.72" x2="12.7" y2="45.72" width="0.1524" layer="91"/>
 </segment>
 </net>
@@
 <pinref part="R1" gate="G$1" pin="2"/>
 <pinref part="U$2" gate="G$1" pin="1"/>
-<wire x1="10.16" y1="81.28" x2="22.86" y2="81.28" width="0.1524" layer="91"/>
-<wire x1="22.86" y1="81.28" x2="22.86" y2="71.12" width="0.1524" layer="91"/>
+<wire x1="10.16" y1="86.36" x2="22.86" y2="86.36" width="0.1524" layer="91"/>
+<wire x1="22.86" y1="86.36" x2="22.86" y2="71.12" width="0.1524" layer="91"/>
 </segment>
 </net>
@@
 <segment>
 <pinref part="R1" gate="G$1" pin="1"/>
-<wire x1="0" y1="81.28" x2="-10.16" y2="81.28" width="0.1524" layer="91"/>
-<wire x1="-10.16" y1="81.28" x2="-10.16" y2="50.8" width="0.1524" layer="91"/>
+<wire x1="0" y1="86.36" x2="-7.62" y2="86.36" width="0.1524" layer="91"/>
+<wire x1="-7.62" y1="86.36" x2="-7.62" y2="50.8" width="0.1524" layer="91"/>
 <pinref part="JP2" gate="A" pin="5"/>
-<wire x1="-10.16" y1="50.8" x2="-15.24" y2="50.8" width="0.1524" layer="91"/>
+<wire x1="-7.62" y1="50.8" x2="-12.7" y2="50.8" width="0.1524" layer="91"/>
 </segment>
 </net>
@@
 <segment>
 <pinref part="JP2" gate="A" pin="4"/>
-<wire x1="-15.24" y1="48.26" x2="-7.62" y2="48.26" width="0.1524" layer="91"/>
+<wire x1="-12.7" y1="48.26" x2="-5.08" y2="48.26" width="0.1524" layer="91"/>
 <pinref part="R2" gate="G$1" pin="1"/>
-<wire x1="-7.62" y1="48.26" x2="-7.62" y2="76.2" width="0.1524" layer="91"/>
-<wire x1="-7.62" y1="76.2" x2="0" y2="76.2" width="0.1524" layer="91"/>
+<wire x1="-5.08" y1="48.26" x2="-5.08" y2="78.74" width="0.1524" layer="91"/>
+<wire x1="-5.08" y1="78.74" x2="0" y2="78.74" width="0.1524" layer="91"/>
 </segment>
 </net>
@@
 <segment>
 <pinref part="R3" gate="G$1" pin="1"/>
-<wire x1="0" y1="71.12" x2="-5.08" y2="71.12" width="0.1524" layer="91"/>
-<wire x1="-5.08" y1="71.12" x2="-5.08" y2="45.72" width="0.1524" layer="91"/>
+<wire x1="0" y1="71.12" x2="-2.54" y2="71.12" width="0.1524" layer="91"/>
+<wire x1="-2.54" y1="71.12" x2="-2.54" y2="45.72" width="0.1524" layer="91"/>
 <pinref part="JP2" gate="A" pin="3"/>
-<wire x1="-5.08" y1="45.72" x2="-15.24" y2="45.72" width="0.1524" layer="91"/>
+<wire x1="-2.54" y1="45.72" x2="-12.7" y2="45.72" width="0.1524" layer="91"/>
 </segment>
 </net>
+<net name="VDD" class="0">
+<segment>
+<pinref part="JP3" gate="A" pin="4"/>
+<wire x1="35.56" y1="43.18" x2="27.94" y2="43.18" width="0.1524" layer="91"/>
+</segment>
+</net>
