File: hw/eagle/projects/size_M/D_ext_power/M_D_ext_power_old.sch (EAGLE design)
At the start: 20 parts

Commit message: pcb M.1 -not finished
Parts:
- removed D.C1: 100n, rcl:C-EUC0603
- removed D.IC2: INA219AIDR, SamacSys_Parts:INA219AIDR
- removed D.R8: 0.1, rcl:R-EU_R0805
- added D.R1: 3k3, rcl:R-EU_R0603
- added D.R2, D.R5: 100k, rcl:R-EU_R0603
- D.C7: value 22u -> 10u; device rcl:C-EUC0805 -> rcl:C-EUC0603
- D.R3: value 12k -> 22k
- D.R6: value 2k2 -> 150
Connections:
- removed net N$13: D.C6.2, D.IC2.IN-, D.LIPOL.2, D.R8.2, D.U1.VBAT
- removed net P0: D.IC2.A1, D.J2.4
- removed net P1: D.IC2.A0, D.J2.3
- removed net P4: D.J2.5, D.R6.1, D.U1.STAT
- removed net SCL: D.IC2.SCL, D.J2.1
- removed net SDA: D.IC2.SDA, D.J2.2
- new net N$1: D.ON/OFF/RESET.P$2, D.ON/OFF/RESET.P$3, D.R1.1
- new net N$20: D.J2.4, D.ON/OFF/RESET.P$1, D.R7.2, D.U2.N_SHDN
- new net PA7: D.J2.3, D.R6.1, D.U1.STAT
- net GND: now also D.R1.2, D.R5.1; no longer D.C1.1, D.IC2.GND, D.ON/OFF/RESET.P$2, D.ON/OFF/RESET.P$3
- net N$5: now also D.J2.5, D.R2.1, D.R5.2; no longer D.ON/OFF/RESET.P$1, D.R7.2, D.U2.N_SHDN
- net N$8: now also D.C6.2, D.LIPOL.2, D.R2.2, D.U1.VBAT; no longer D.IC2.IN+, D.R8.1
- net VDD: no longer D.C1.2, D.IC2.VS
Other:
- moved on the sheet: D.C7, D.J2, D.J3, D.L1, D.LIPOL, D.R4, D.R7, D.T1, D.U2, U$1
