File: pcb/eagle/projects/size_M/A_base/M_A_base.sch (EAGLE design)
At the start: 16 parts

Commit message: PCB M.1
Parts:
- added JP1, JP2, JP3, JP4: (no value), pinhead2:PINHD-1X2
Connections:
- new net VBAT: JP1.2, JP2.2, JP3.2, JP4.2
- new net VUSB: JP1.1, JP2.1, JP3.1, JP4.1
Changed lines of the file:
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@@
 <part name="A.J15" library="pinhead2" deviceset="PINHD-1X4" device="" package3d_urn="urn:adsk.eagle:package:22407/2"/>
 <part name="A.J16" library="pinhead2" deviceset="PINHD-1X4" device="" package3d_urn="urn:adsk.eagle:package:22407/2"/>
+<part name="JP1" library="pinhead2" deviceset="PINHD-1X2" device="" package3d_urn="urn:adsk.eagle:package:22435/2"/>
+<part name="JP2" library="pinhead2" deviceset="PINHD-1X2" device="" package3d_urn="urn:adsk.eagle:package:22435/2"/>
+<part name="JP3" library="pinhead2" deviceset="PINHD-1X2" device="" package3d_urn="urn:adsk.eagle:package:22435/2"/>
+<part name="JP4" library="pinhead2" deviceset="PINHD-1X2" device="" package3d_urn="urn:adsk.eagle:package:22435/2"/>
 </parts>
 <sheets>
@@
 <attribute name="NAME" x="115.57" y="-14.605" size="1.778" layer="95"/>
 <attribute name="VALUE" x="115.57" y="-30.48" size="1.778" layer="96"/>
+</instance>
+<instance part="JP1" gate="G$1" x="-25.4" y="10.16" smashed="yes" rot="R90">
+<attribute name="NAME" x="-31.115" y="3.81" size="1.778" layer="95" rot="R90"/>
+<attribute name="VALUE" x="-20.32" y="3.81" size="1.778" layer="96" rot="R90"/>
+</instance>
+<instance part="JP2" gate="G$1" x="12.7" y="10.16" smashed="yes" rot="R90">
+<attribute name="NAME" x="6.985" y="3.81" size="1.778" layer="95" rot="R90"/>
+<attribute name="VALUE" x="17.78" y="3.81" size="1.778" layer="96" rot="R90"/>
+</instance>
+<instance part="JP3" gate="G$1" x="53.34" y="10.16" smashed="yes" rot="R90">
+<attribute name="NAME" x="47.625" y="3.81" size="1.778" layer="95" rot="R90"/>
+<attribute name="VALUE" x="58.42" y="3.81" size="1.778" layer="96" rot="R90"/>
+</instance>
+<instance part="JP4" gate="G$1" x="91.44" y="10.16" smashed="yes" rot="R90">
+<attribute name="NAME" x="85.725" y="3.81" size="1.778" layer="95" rot="R90"/>
+<attribute name="VALUE" x="96.52" y="3.81" size="1.778" layer="96" rot="R90"/>
 </instance>
 </instances>
@@
 </segment>
 </net>
+<net name="VBAT" class="0">
+<segment>
+<pinref part="JP1" gate="G$1" pin="2"/>
+<wire x1="-25.4" y1="7.62" x2="-25.4" y2="2.54" width="0.1524" layer="91"/>
+<pinref part="JP2" gate="G$1" pin="2"/>
+<wire x1="-25.4" y1="2.54" x2="12.7" y2="2.54" width="0.1524" layer="91"/>
+<wire x1="12.7" y1="2.54" x2="12.7" y2="7.62" width="0.1524" layer="91"/>
+<pinref part="JP3" gate="G$1" pin="2"/>
+<wire x1="12.7" y1="2.54" x2="53.34" y2="2.54" width="0.1524" layer="91"/>
+<wire x1="53.34" y1="2.54" x2="53.34" y2="7.62" width="0.1524" layer="91"/>
+<junction x="12.7" y="2.54"/>
+<pinref part="JP4" gate="G$1" pin="2"/>
+<wire x1="53.34" y1="2.54" x2="91.44" y2="2.54" width="0.1524" layer="91"/>
+<wire x1="91.44" y1="2.54" x2="91.44" y2="7.62" width="0.1524" layer="91"/>
+<junction x="53.34" y="2.54"/>
+</segment>
+</net>
+<net name="VUSB" class="0">
+<segment>
+<pinref part="JP4" gate="G$1" pin="1"/>
+<wire x1="88.9" y1="7.62" x2="88.9" y2="0" width="0.1524" layer="91"/>
+<wire x1="88.9" y1="0" x2="50.8" y2="0" width="0.1524" layer="91"/>
+<pinref part="JP3" gate="G$1" pin="1"/>
+<wire x1="50.8" y1="0" x2="50.8" y2="7.62" width="0.1524" layer="91"/>
+<pinref part="JP2" gate="G$1" pin="1"/>
+<wire x1="50.8" y1="0" x2="10.16" y2="0" width="0.1524" layer="91"/>
+<wire x1="10.16" y1="0" x2="10.16" y2="7.62" width="0.1524" layer="91"/>
+<junction x="50.8" y="0"/>
+<pinref part="JP1" gate="G$1" pin="1"/>
+<wire x1="10.16" y1="0" x2="-27.94" y2="0" width="0.1524" layer="91"/>
+<wire x1="-27.94" y1="0" x2="-27.94" y2="7.62" width="0.1524" layer="91"/>
+<junction x="10.16" y="0"/>
+</segment>
+</net>

Commit message: updated PCBs after delivery of v1
Parts:
- removed A.J16: (no value), pinhead2:PINHD-1X4
Connections:
- net GND: no longer A.J16.3
- net SCL: no longer A.J16.1
- net SDA: no longer A.J16.2
- net VCC: no longer A.J16.4
Changed lines of the file:
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@@
 <part name="A.J14" library="pinhead2" deviceset="PINHD-1X2" device="/90" package3d_urn="urn:adsk.eagle:package:22437/2"/>
 <part name="A.J15" library="pinhead2" deviceset="PINHD-1X4" device="" package3d_urn="urn:adsk.eagle:package:22407/2"/>
-<part name="A.J16" library="pinhead2" deviceset="PINHD-1X4" device="" package3d_urn="urn:adsk.eagle:package:22407/2"/>
 <part name="JP1" library="pinhead2" deviceset="PINHD-1X2" device="" package3d_urn="urn:adsk.eagle:package:22435/2"/>
 <part name="JP2" library="pinhead2" deviceset="PINHD-1X2" device="" package3d_urn="urn:adsk.eagle:package:22435/2"/>
@@
 <attribute name="NAME" x="-46.99" y="-28.575" size="1.778" layer="95" rot="R180"/>
 <attribute name="VALUE" x="-46.99" y="-12.7" size="1.778" layer="96" rot="R180"/>
-</instance>
-<instance part="A.J16" gate="A" x="121.92" y="-22.86" smashed="yes">
-<attribute name="NAME" x="115.57" y="-14.605" size="1.778" layer="95"/>
-<attribute name="VALUE" x="115.57" y="-30.48" size="1.778" layer="96"/>
 </instance>
 <instance part="JP1" gate="G$1" x="-25.4" y="10.16" smashed="yes" rot="R90">
@@
 <pinref part="A.J15" gate="A" pin="1"/>
 <wire x1="-25.4" y1="-25.4" x2="-50.8" y2="-25.4" width="0.1524" layer="91"/>
-<pinref part="A.J16" gate="A" pin="4"/>
-<wire x1="119.38" y1="-25.4" x2="93.98" y2="-25.4" width="0.1524" layer="91"/>
 </segment>
 </net>
@@
 <wire x1="-33.02" y1="-22.86" x2="-50.8" y2="-22.86" width="0.1524" layer="91"/>
 <junction x="-33.02" y="-22.86"/>
-<wire x1="96.52" y1="-43.18" x2="101.6" y2="-43.18" width="0.1524" layer="91"/>
-<junction x="96.52" y="-43.18"/>
-<wire x1="101.6" y1="-43.18" x2="101.6" y2="-22.86" width="0.1524" layer="91"/>
-<pinref part="A.J16" gate="A" pin="3"/>
-<wire x1="101.6" y1="-22.86" x2="119.38" y2="-22.86" width="0.1524" layer="91"/>
 </segment>
 </net>
@@
 <junction x="91.44" y="-5.08"/>
 <pinref part="A.J12" gate="A" pin="7"/>
-<wire x1="104.14" y1="-5.08" x2="104.14" y2="-17.78" width="0.1524" layer="91"/>
-<wire x1="104.14" y1="-17.78" x2="104.14" y2="-20.32" width="0.1524" layer="91"/>
+<wire x1="104.14" y1="-5.08" x2="104.14" y2="-20.32" width="0.1524" layer="91"/>
 <wire x1="104.14" y1="-20.32" x2="96.52" y2="-20.32" width="0.1524" layer="91"/>
 <wire x1="104.14" y1="-20.32" x2="104.14" y2="-45.72" width="0.1524" layer="91"/>
@@
 <wire x1="-35.56" y1="-17.78" x2="-50.8" y2="-17.78" width="0.1524" layer="91"/>
 <junction x="-35.56" y="-17.78"/>
-<pinref part="A.J16" gate="A" pin="1"/>
-<wire x1="104.14" y1="-17.78" x2="119.38" y2="-17.78" width="0.1524" layer="91"/>
-<junction x="104.14" y="-17.78"/>
 </segment>
 </net>
@@
 <junction x="93.98" y="-2.54"/>
 <pinref part="A.J11" gate="A" pin="8"/>
-<wire x1="106.68" y1="-2.54" x2="106.68" y2="-20.32" width="0.1524" layer="91"/>
-<wire x1="106.68" y1="-20.32" x2="106.68" y2="-30.48" width="0.1524" layer="91"/>
+<wire x1="106.68" y1="-2.54" x2="106.68" y2="-30.48" width="0.1524" layer="91"/>
 <wire x1="106.68" y1="-30.48" x2="96.52" y2="-30.48" width="0.1524" layer="91"/>
 <junction x="78.74" y="-2.54"/>
@@
 <pinref part="A.J15" gate="A" pin="3"/>
 <wire x1="-38.1" y1="-20.32" x2="-50.8" y2="-20.32" width="0.1524" layer="91"/>
-<pinref part="A.J16" gate="A" pin="2"/>
-<wire x1="119.38" y1="-20.32" x2="106.68" y2="-20.32" width="0.1524" layer="91"/>
-<junction x="106.68" y="-20.32"/>
 </segment>
 </net>
