File: pcb/eagle/projects/size_M/3x4/M_3x4._v3.brd (EAGLE design)
At the start: 100 x 76 mm, 140 parts, among them P1 TPB1,27, U1 CP2104-F03-GM

Commit message: PCB M.3
Parts:
- removed JP10: (no value), pinhead2:1X08
- removed JP12, JP13: (no value), pinhead2:1X06
- removed JP14: (no value), pinhead2:1X05
- removed K.R6: 0R, rcl:R0603
- removed U$13, U$14, U$15, U$16, U$17, U$18, U$19, U$20: PINHD-1X5_AUTO, pinhead2:1X5_AUTO
- added D.R4, I.R5: 100k, rcl:R0603
- added D.T2: FDV304, !stavebnice03:SOT23
- added G.J4: (no value), pinhead2:1X06
- added G.J5: (no value), pinhead2:1X04
- added I.T1: (no value), !stavebnice03:SOT23
- added L.C1: 100n, rcl:C0603
- added L.R1, L.R2: 1k, rcl:R0603
- added L.R3, L.R4, L.R5, L.R6: 2k2, rcl:R0603
- added L.SW1: 5_WAY_SWITCH, hugo:5_WAY_SWITCH
- D.D2: value SHOTKY -> SHOTKY_2.8; device hugo:SHOTKY -> hugo:SHOTKY_2.8
- JP7: device pinhead2:1X06 -> pinhead2:1X08
- JP8: device pinhead2:1X05 -> pinhead2:1X06
- U$11: value MICRO_SD -> PINHD-1X5_AUTO; device hugo:MOCRO_SD -> pinhead2:1X5_AUTO
- U$12: value BUTTON-SWITCH -> PINHD-1X5_AUTO; device hugo:BUTTON-SWITCH -> pinhead2:1X5_AUTO
- U$3: value PINHD-1X5_AUTO -> BUTTON-SWITCH; device pinhead2:1X5_AUTO -> hugo:BUTTON-SWITCH
- U$4: value PINHD-1X5_AUTO -> MICRO_SD; device pinhead2:1X5_AUTO -> hugo:MOCRO_SD
- moved U$4 80.5 mm to (4.40, 30.6), flipped to the bottom, turned to 180 degrees
- moved I.J1 53.7 mm to (21.1, 36.0)
- moved JP8 35.6 mm to (66.6, 60.0), turned to 90 degrees
- moved I.J3 33.9 mm to (69.1, 60.0)
- moved JP6 33.9 mm to (50.9, 62.5)
- moved U$12 31.7 mm to (60.0, 27.1), turned to 0 degrees
- moved U$11 31.6 mm to (60.0, 29.6), flipped to the top, turned to 0 degrees
- moved JP7 31.0 mm to (54.0, 60.0)
- moved U$3 27.7 mm to (60.0, 58.7), turned to 90 degrees
- moved I.C2 27.3 mm to (15.5, 39.1)
- moved I.R6 27.1 mm to (13.1, 43.5)
- moved U$6 24.5 mm to (60.0, 42.4)
- moved U$9 24.5 mm to (60.0, 34.7)
- moved U$8 24.5 mm to (60.0, 37.3)
- moved U$5 24.5 mm to (60.0, 44.9)
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Connections:
- removed net N$23: JP6.2, JP7.2
- removed net N$24 (its old number): JP6.1, JP7.1
- removed net N$26: JP11.2, JP8.2
- new net N$41: L.R2.1, L.R3.2, L.SW1.6
- new net VCC6: G.J5.3, L.C1.2, L.R6.2
- net GND2: now also D.R4.2
- net GND3: now also I.J3.4, JP7.2, JP8.2, K.C1.2, K.C2.2, K.U1.GND, U$3.P$1, U$3.P$2; no longer JP11.4, JP7.6, JP8.4
- net GND4: now also H.J4.4, I.C1.2, I.C2.1, I.C4.1, I.C5.1, I.J1.4, I.J2.6, I.R6.1, I.U1.3, I.U1.6, I.U2.7, I.U2.9, I.U2.P$10, I.U2.P$11, I.U2.P$12, I.U2.P$13, U$4.6, U$4.G1, U$4.G2, U$4.G3, U$4.G4; no longer G.C2.1, G.C4.1, G.C5.1, G.J1.6, G.J2.4, G.J3.$1, G.J3.$2, G.J3.6, G.MOTO1.$1, G.MOTO1.$2, G.MOTO1.6, G.U1.14, G.U2.10, G.U2.11, G.U2.14, G.U2.15
- net GND5: now also G.C2.1, G.C4.1, G.C5.1, G.J1.6, G.J2.4, G.J3.$1, G.J3.$2, G.J3.6, G.MOTO1.$1, G.MOTO1.$2, G.MOTO1.6, G.U1.14, G.U2.10, G.U2.11, G.U2.14, G.U2.15; no longer H.J4.4, I.C1.2, I.C2.1, I.C4.1, I.C5.1, I.J2.6, I.J3.4, I.R6.1, I.U1.3, I.U1.6, I.U2.7, I.U2.9, I.U2.P$10, I.U2.P$11, I.U2.P$12, I.U2.P$13, U$11.6, U$11.G1, U$11.G2, U$11.G3, U$11.G4
- net GND6: now also G.J4.6, G.J5.4, L.C1.1, L.R1.2, L.SW1.4; no longer I.J1.4, JP10.2, JP12.2, JP9.6, K.C1.2, K.C2.2, K.U1.GND, U$12.P$1, U$12.P$2
- net GND8: now also JP11.4, JP9.6; no longer JP13.6, JP14.4
- net N$20: now also D.J2.5, D.T2.D; no longer JP6.5, JP7.5
- net N$21: now also JP6.2, JP8.4; no longer JP6.4
- net N$22: now also JP6.1, JP8.3; no longer JP6.3
- net N$25: now also JP6.5, JP8.6, K.D1.C, K.R3.1, K.R4.1, K.U1.OUT; no longer JP11.5, JP8.5
- net N$27: now also JP6.3, JP7.5, JP8.5, K.R1.2, U$3.P$3; no longer JP11.1, JP8.1
- net N$28: now also JP6.4, JP7.8, K.R5.1; no longer JP11.3, JP8.3
- net N$38: now also I.R5.1, I.T1.G
- net N$39: now also I.C4.2, I.J1.3, I.R5.2, I.T1.S; no longer JP10.4, JP12.4, JP9.2
- net N$40: now also L.R1.1, L.R2.2, L.SW1.5; no longer JP10.3, JP12.3, JP9.1
- net N$42: now also L.R3.1, L.R4.2, L.SW1.3; no longer JP12.6, JP9.5, K.D1.C, K.R3.1, K.R4.1, K.U1.OUT
- net N$43: now also L.R5.2, L.SW1.2; no longer JP10.5, JP12.5, JP9.3, K.R1.2, K.R6.1, U$12.P$3
- net N$44: now also G.J4.5, L.R6.1, L.SW1.1; no longer JP10.8, JP9.4, K.R5.1
- net N$45: now also L.R4.1, L.R5.1; no longer JP10.6, K.R4.2
- net N$46: now also U$5.1, U$5.2, U$5.3, U$5.4, U$5.5; no longer JP10.7, K.R3.2, K.R5.2
- net N$47: now also U$6.1, U$6.2, U$6.3, U$6.4, U$6.5; no longer I.J1.2, K.R6.2
- net N$48: now also U$7.1, U$7.2, U$7.3, U$7.4, U$7.5; no longer U$13.1, U$13.2, U$13.3, U$13.4, U$13.5
- net N$49: now also U$8.1, U$8.2, U$8.3, U$8.4, U$8.5; no longer U$14.1, U$14.2, U$14.3, U$14.4, U$14.5
- net N$50: now also U$9.1, U$9.2, U$9.3, U$9.4, U$9.5; no longer U$15.1, U$15.2, U$15.3, U$15.4, U$15.5
- net N$51: now also U$10.1, U$10.2, U$10.3, U$10.4, U$10.5; no longer U$16.1, U$16.2, U$16.3, U$16.4, U$16.5
- net N$52: now also U$11.1, U$11.2, U$11.3, U$11.4, U$11.5; no longer U$17.1, U$17.2, U$17.3, U$17.4, U$17.5
- net N$53: now also U$12.1, U$12.2, U$12.3, U$12.4, U$12.5; no longer U$18.1, U$18.2, U$18.3, U$18.4, U$18.5
- net N$54: now also JP7.6, K.R4.2; no longer U$19.1, U$19.2, U$19.3, U$19.4, U$19.5
- net N$55: now also JP7.7, K.R3.2, K.R5.2; no longer U$20.1, U$20.2, U$20.3, U$20.4, U$20.5
- net PA3: now also D.T2.S; no longer D.J2.5
- net SDCLK: now also U$4.5; no longer U$11.5
- net SDCMD: now also U$4.3; no longer U$11.3
- net SDDAT: now also U$4.7; no longer U$11.7
- net VCC2: now also D.R4.1, D.T2.G
- net VCC3: now also I.J3.3, JP7.1, JP8.1, K.C1.1, K.C2.1, K.R1.1, K.R2.1, K.U1.VCC; no longer G.C2.2, G.C5.2, G.J2.3, G.U1.1, G.U2.1, G.U2.5
- net VCC4: now also I.T1.D, U$4.4; no longer I.C4.2, I.J3.3, U$11.4
- net VCC5: now also G.C2.2, G.C5.2, G.J2.3, G.U1.1, G.U2.1, G.U2.5; no longer I.J1.3, JP10.1, JP12.1, K.C1.1, K.C2.1, K.R1.1, K.R2.1, K.U1.VCC
- net VDD: now also JP11.3; no longer JP14.3
Routing:
- net GND3: track 0.00 -> 54.7 mm, vias 0 -> 3
- net N$25: track 1.54 -> 33.3 mm, vias 0 -> 1
- net N$27: track 1.52 -> 27.1 mm, vias 0 -> 1
- net N$43: track 30.8 -> 6.62 mm, vias 1 -> 0
- net VCC2: track 22.1 -> 43.4 mm, vias 1 -> 3
- net N$42: track 33.4 -> 14.2 mm, vias 1 -> 0
- net VCC6: track 0.00 -> 18.8 mm
- net N$38: track 0.00 -> 18.4 mm, vias 0 -> 2
- net N$41: track 0.00 -> 15.7 mm
- net N$22: track 1.53 -> 16.8 mm
- net N$21: track 1.55 -> 16.8 mm
- net N$20: track 1.56 -> 16.1 mm
- net GND2: track 142.6 -> 128.5 mm, vias 6 -> 3
- net GND4: track 93.8 -> 103.6 mm, vias 7 -> 3
- net GND6: track 54.7 -> 45.2 mm, vias 4 -> 2
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Other:
- board text added: "5wSwitch M3"
- board text added: "Hugo M3"
- board text added: "sensor M.3"
- board text removed: "M.3"
- board text removed: "M.3 sensor"
- board text removed: "proto"
