File: pcb/eagle/projects/size_M/3x4/M_3x4._v4.brd (EAGLE design)
At the start: 100 x 76 mm, 123 parts, among them J1 RJ11, P1 TPB1,27, U1 CP2104-F03-GM

Commit message: PCB v4
Other:
- outline, holes or cut-outs redrawn
