File: pcb/eagle/projects/size_M/E_ext_proto/M_E_ext_proto.sch (EAGLE design)
At the start: 12 parts

Commit message: PCB's adjustments + sensor extension
Connections:
- removed net VDD: JP11.4, JP3.4
- new net N$10: JP11.3, JP3.3
- net GND: now also JP11.4, JP3.4; no longer JP11.3, JP3.3
Changed lines of the file:
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@@
 <net name="GND" class="0">
 <segment>
-<wire x1="114.3" y1="35.56" x2="121.92" y2="35.56" width="0.1524" layer="91"/>
-<pinref part="JP11" gate="A" pin="3"/>
-<pinref part="JP3" gate="A" pin="3"/>
-<wire x1="114.3" y1="35.56" x2="109.22" y2="35.56" width="0.1524" layer="91"/>
-<junction x="114.3" y="35.56"/>
 <pinref part="JP2" gate="A" pin="6"/>
 <wire x1="78.74" y1="38.1" x2="73.66" y2="38.1" width="0.1524" layer="91"/>
@@
 <wire x1="78.74" y1="38.1" x2="78.74" y2="48.26" width="0.1524" layer="91"/>
 <wire x1="78.74" y1="48.26" x2="109.22" y2="48.26" width="0.1524" layer="91"/>
-<wire x1="109.22" y1="48.26" x2="109.22" y2="35.56" width="0.1524" layer="91"/>
-</segment>
-</net>
-<net name="VDD" class="0">
-<segment>
-<wire x1="121.92" y1="33.02" x2="114.3" y2="33.02" width="0.1524" layer="91"/>
+<wire x1="109.22" y1="48.26" x2="109.22" y2="33.02" width="0.1524" layer="91"/>
 <pinref part="JP11" gate="A" pin="4"/>
 <pinref part="JP3" gate="A" pin="4"/>
+<wire x1="121.92" y1="33.02" x2="114.3" y2="33.02" width="0.1524" layer="91"/>
 <wire x1="114.3" y1="33.02" x2="109.22" y2="33.02" width="0.1524" layer="91"/>
 <junction x="114.3" y="33.02"/>
@@
 </segment>
 </net>
+<net name="N$10" class="0">
+<segment>
+<pinref part="JP11" gate="A" pin="3"/>
+<wire x1="114.3" y1="35.56" x2="121.92" y2="35.56" width="0.1524" layer="91"/>
+<pinref part="JP3" gate="A" pin="3"/>
+</segment>
+</net>

Commit message: reorganized pcb folders
Connections:
- new net N$9: JP1.6, JP2.6
- net GND: no longer JP1.6, JP2.6
Changed lines of the file:
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@@
 <net name="GND" class="0">
 <segment>
-<pinref part="JP2" gate="A" pin="6"/>
-<wire x1="78.74" y1="38.1" x2="73.66" y2="38.1" width="0.1524" layer="91"/>
-<pinref part="JP1" gate="A" pin="6"/>
-<junction x="73.66" y="38.1"/>
-<wire x1="73.66" y1="38.1" x2="66.04" y2="38.1" width="0.1524" layer="91"/>
-<wire x1="78.74" y1="38.1" x2="78.74" y2="48.26" width="0.1524" layer="91"/>
-<wire x1="78.74" y1="48.26" x2="109.22" y2="48.26" width="0.1524" layer="91"/>
-<wire x1="109.22" y1="48.26" x2="109.22" y2="33.02" width="0.1524" layer="91"/>
 <pinref part="JP11" gate="A" pin="4"/>
 <pinref part="JP3" gate="A" pin="4"/>
 <wire x1="121.92" y1="33.02" x2="114.3" y2="33.02" width="0.1524" layer="91"/>
-<wire x1="114.3" y1="33.02" x2="109.22" y2="33.02" width="0.1524" layer="91"/>
-<junction x="114.3" y="33.02"/>
 </segment>
 </net>
@@
 </segment>
 </net>
+<net name="N$9" class="0">
+<segment>
+<pinref part="JP2" gate="A" pin="6"/>
+<pinref part="JP1" gate="A" pin="6"/>
+<wire x1="73.66" y1="38.1" x2="66.04" y2="38.1" width="0.1524" layer="91"/>
+</segment>
+</net>
