File: pcb/eagle/projects/size_M/F_ext_breadboard/M_F_ext_breadboard.sch (EAGLE design)
At the start: 10 parts

Commit message: reorganized pcb folders
Connections:
- net GND: no longer JP2.6
Changed lines of the file:
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@@
 <net name="GND" class="0">
 <segment>
-<wire x1="73.66" y1="50.8" x2="109.22" y2="50.8" width="0.1524" layer="91"/>
-<pinref part="JP2" gate="A" pin="6"/>
-<wire x1="73.66" y1="50.8" x2="73.66" y2="38.1" width="0.1524" layer="91"/>
-<wire x1="73.66" y1="38.1" x2="66.04" y2="38.1" width="0.1524" layer="91"/>
 <pinref part="JP11" gate="A" pin="4"/>
-<wire x1="109.22" y1="50.8" x2="109.22" y2="33.02" width="0.1524" layer="91"/>
 <wire x1="109.22" y1="33.02" x2="121.92" y2="33.02" width="0.1524" layer="91"/>
 </segment>
