File: pcb/eagle/projects/size_M/J_ext_disp/M_J_ext_disp.brd (EAGLE design)
At the start: 11 parts, among them J1 SSD_1306_STM32_OLED

Commit message: PCB M.1
Parts:
- removed JP2: (no value), pinhead2:1X03
- added I.J2: (no value), pinhead2:1X02
- renumbered H.C1 to J.C1, H.C2 to J.C2, H.C3 to J.C3, H.C4 to J.C4, H.C5 to J.C5, H.C6 to J.C6, H.R1 to J.R1, H.R2 to J.R2, J1 to I.J3, JP1 to J.J1
Connections:
- net GND: now also I.J2.2; no longer JP2.2
- net VDD: now also I.J2.1; no longer JP2.1
Routing:
- net GND: track 72.2 -> 70.9 mm
- net VDD: track 27.6 -> 26.4 mm

Commit message: updated PCBs for version 2
Parts:
- added J.C7: 2u2, rcl:C0603
- added J.R3: 2k2, rcl:R0603
- moved J.R2 6.42 mm to (13.1, 5.33), turned to 90 degrees
- moved J.C6 5.95 mm to (15.2, 5.33)
- moved J.C5 5.86 mm to (17.3, 5.33)
- moved J.C4 0.61 mm to (15.2, 9.14)
- moved J.C1 0.54 mm to (17.3, 9.14)
- moved J.R1 0.47 mm to (7.95, 9.14), turned to 270 degrees
- moved J.C2 0.43 mm to (5.82, 9.14)
- moved J.C3 0.42 mm to (3.66, 9.14)
Connections:
- new net N$2: I.J3.P$12, J.C7.2, J.R3.2
- net GND: now also J.C7.1
- net VDD: now also J.R3.1; no longer I.J3.P$12
Routing:
- net N$2: track 0.00 -> 9.57 mm
- net PA7: track 13.1 -> 22.3 mm
- net GND: track 70.9 -> 79.9 mm
- net VDD: track 26.4 -> 22.6 mm
- net N$7: track 7.82 -> 6.89 mm
- net N$1: track 6.73 -> 7.40 mm
- net N$10: track 5.44 -> 4.82 mm
- net N$8: track 5.09 -> 4.51 mm
- net N$9: track 7.81 -> 7.29 mm
Other:
- board text added: "disp M.2"
- board text removed: "disp M.1"

Commit message: PCB v7 * 14 pin attiny is main adapter chip now. * changed adapter pin meaning (a1-a5, swapped RX-TX, VUSB replaced by A5, top most pin changed from GND to A4) * changed usb chip of main board
Changed lines of the file:
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@@
 <setting verticaltext="up"/>
 </settings>
-<grid distance="1" unitdist="mil" unit="mil" style="lines" multiple="1" display="yes" altdistance="0.1" altunitdist="mm" altunit="mm"/>
+<grid distance="1" unitdist="mil" unit="mm" style="lines" multiple="1" display="yes" altdistance="0.1" altunitdist="mm" altunit="mm"/>
 <layers>
-<layer number="1" name="Top" color="4" fill="1" visible="no" active="yes"/>
-<layer number="16" name="Bottom" color="1" fill="1" visible="no" active="yes"/>
+<layer number="1" name="Top" color="4" fill="1" visible="yes" active="yes"/>
+<layer number="16" name="Bottom" color="1" fill="1" visible="yes" active="yes"/>
 <layer number="17" name="Pads" color="2" fill="1" visible="yes" active="yes"/>
 <layer number="18" name="Vias" color="2" fill="1" visible="yes" active="yes"/>
-<layer number="19" name="Unrouted" color="6" fill="1" visible="no" active="yes"/>
-<layer number="20" name="Dimension" color="24" fill="1" visible="no" active="yes"/>
-<layer number="21" name="tPlace" color="23" fill="1" visible="no" active="yes"/>
+<layer number="19" name="Unrouted" color="6" fill="1" visible="yes" active="yes"/>
+<layer number="20" name="Dimension" color="24" fill="1" visible="yes" active="yes"/>
+<layer number="21" name="tPlace" color="23" fill="1" visible="yes" active="yes"/>
 <layer number="22" name="bPlace" color="47" fill="1" visible="yes" active="yes"/>
-<layer number="23" name="tOrigins" color="15" fill="1" visible="no" active="yes"/>
+<layer number="23" name="tOrigins" color="15" fill="1" visible="yes" active="yes"/>
 <layer number="24" name="bOrigins" color="15" fill="1" visible="yes" active="yes"/>
-<layer number="25" name="tNames" color="7" fill="1" visible="no" active="yes"/>
+<layer number="25" name="tNames" color="7" fill="1" visible="yes" active="yes"/>
 <layer number="26" name="bNames" color="7" fill="1" visible="yes" active="yes"/>
 <layer number="27" name="tValues" color="7" fill="1" visible="no" active="yes"/>
 <layer number="28" name="bValues" color="7" fill="1" visible="no" active="yes"/>
 <layer number="29" name="tStop" color="7" fill="3" visible="no" active="yes"/>
-<layer number="30" name="bStop" color="7" fill="6" visible="yes" active="yes"/>
+<layer number="30" name="bStop" color="7" fill="6" visible="no" active="yes"/>
 <layer number="31" name="tCream" color="7" fill="4" visible="no" active="yes"/>
 <layer number="32" name="bCream" color="7" fill="5" visible="no" active="yes"/>
@@
 <layer number="37" name="tTest" color="7" fill="1" visible="no" active="yes"/>
 <layer number="38" name="bTest" color="7" fill="1" visible="no" active="yes"/>
-<layer number="39" name="tKeepout" color="4" fill="11" visible="no" active="yes"/>
-<layer number="40" name="bKeepout" color="1" fill="11" visible="no" active="yes"/>
-<layer number="41" name="tRestrict" color="4" fill="10" visible="no" active="yes"/>
-<layer number="42" name="bRestrict" color="1" fill="10" visible="no" active="yes"/>
+<layer number="39" name="tKeepout" color="4" fill="11" visible="yes" active="yes"/>
+<layer number="40" name="bKeepout" color="1" fill="11" visible="yes" active="yes"/>
+<layer number="41" name="tRestrict" color="4" fill="10" visible="yes" active="yes"/>
+<layer number="42" name="bRestrict" color="1" fill="10" visible="yes" active="yes"/>
 <layer number="43" name="vRestrict" color="2" fill="10" visible="no" active="yes"/>
 <layer number="44" name="Drills" color="7" fill="1" visible="no" active="yes"/>
@@
 <layer number="46" name="Milling" color="3" fill="1" visible="no" active="yes"/>
 <layer number="47" name="Measures" color="7" fill="1" visible="no" active="yes"/>
-<layer number="48" name="Document" color="8" fill="1" visible="yes" active="yes"/>
+<layer number="48" name="Document" color="8" fill="1" visible="no" active="yes"/>
 <layer number="49" name="Reference" color="7" fill="1" visible="no" active="yes"/>
 <layer number="50" name="dxf" color="7" fill="1" visible="no" active="no"/>
-<layer number="51" name="tDocu" color="7" fill="1" visible="no" active="yes"/>
-<layer number="52" name="bDocu" color="7" fill="1" visible="no" active="yes"/>
+<layer number="51" name="tDocu" color="7" fill="1" visible="yes" active="yes"/>
+<layer number="52" name="bDocu" color="7" fill="1" visible="yes" active="yes"/>
 <layer number="53" name="tGND_GNDA" color="7" fill="9" visible="no" active="no"/>
 <layer number="54" name="bGND_GNDA" color="1" fill="9" visible="no" active="no"/>
@@
 <wire x1="15.3774" y1="16.2066" x2="15.367" y2="16.217" width="0.3048" layer="16"/>
 <wire x1="5.602" y1="14.228" x2="5.602" y2="12.7622" width="0.3048" layer="16"/>
-<polygon width="0.3048" layer="1" isolate="0.3048">
+<polygon width="0.254" layer="1" isolate="0.254">
 <vertex x="0.5" y="20.5"/>
 <vertex x="0.5" y="0.5"/>
@@
 <vertex x="20.5" y="20.5"/>
 </polygon>
-<polygon width="0.3048" layer="16" isolate="0.3048">
+<polygon width="0.254" layer="16" isolate="0.254">
 <vertex x="0.5" y="0.5"/>
 <vertex x="20.5" y="0.5"/>
