File: pcb/eagle/projects/size_M/J_ext_disp/M_J_ext_disp.sch (EAGLE design)
At the start: 11 parts, among them J1 SSD_1306_STM32_OLED

Commit message: PCB M.1
Parts:
- removed JP2: (no value), pinhead2:PINHD-1X3
- added I.J2: (no value), pinhead2:PINHD-1X2
- renumbered H.C1 to J.C1, H.C2 to J.C2, H.C3 to J.C3, H.C4 to J.C4, H.C5 to J.C5, H.C6 to J.C6, H.R1 to J.R1, H.R2 to J.R2, J1 to I.J3, JP1 to J.J1
Connections:
- net GND: now also I.J2.2; no longer JP2.2
- net VDD: now also I.J2.1; no longer JP2.1

Commit message: updated PCBs for version 2
Parts:
- added J.C7: 2u2, rcl:C-EUC0603
- added J.R3: 2k2, rcl:R-EU_R0603
Connections:
- new net N$2: I.J3.RES#, J.C7.2, J.R3.2
- net GND: now also J.C7.1
- net VDD: now also J.R3.1; no longer I.J3.RES#
Changed lines of the file:
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@@
 <part name="J.J1" library="pinhead2" deviceset="PINHD-1X3" device="" package3d_urn="urn:adsk.eagle:package:22458/2"/>
 <part name="I.J2" library="pinhead2" deviceset="PINHD-1X2" device="" package3d_urn="urn:adsk.eagle:package:22435/2"/>
+<part name="J.R3" library="rcl" library_urn="urn:adsk.eagle:library:334" deviceset="R-EU_" device="R0603" package3d_urn="urn:adsk.eagle:package:23555/3" value="2k2"/>
+<part name="J.C7" library="rcl" library_urn="urn:adsk.eagle:library:334" deviceset="C-EU" device="C0603" package3d_urn="urn:adsk.eagle:package:23616/2" value="2u2"/>
 </parts>
 <sheets>
@@
 <attribute name="NAME" x="62.23" y="59.055" size="1.778" layer="95"/>
 <attribute name="VALUE" x="62.23" y="48.26" size="1.778" layer="96"/>
+</instance>
+<instance part="J.R3" gate="G$1" x="7.62" y="127" smashed="yes" rot="R270">
+<attribute name="NAME" x="9.1186" y="130.81" size="1.778" layer="95" rot="R270"/>
+<attribute name="VALUE" x="4.318" y="130.81" size="1.778" layer="96" rot="R270"/>
+</instance>
+<instance part="J.C7" gate="G$1" x="-7.62" y="121.92" smashed="yes" rot="R90">
+<attribute name="NAME" x="-8.001" y="123.444" size="1.778" layer="95" rot="R90"/>
+<attribute name="VALUE" x="-2.921" y="123.444" size="1.778" layer="96" rot="R90"/>
 </instance>
 </instances>
@@
 <wire x1="2.54" y1="137.16" x2="-17.78" y2="137.16" width="0.1524" layer="91"/>
 <junction x="-17.78" y="137.16"/>
-<wire x1="-10.16" y1="132.08" x2="-17.78" y2="132.08" width="0.1524" layer="91"/>
+<wire x1="-10.16" y1="132.08" x2="-12.7" y2="132.08" width="0.1524" layer="91"/>
 <junction x="-17.78" y="132.08"/>
+<pinref part="J.C7" gate="G$1" pin="1"/>
+<wire x1="-12.7" y1="132.08" x2="-17.78" y2="132.08" width="0.1524" layer="91"/>
+<wire x1="-10.16" y1="121.92" x2="-12.7" y2="121.92" width="0.1524" layer="91"/>
+<wire x1="-12.7" y1="121.92" x2="-12.7" y2="132.08" width="0.1524" layer="91"/>
+<junction x="-12.7" y="132.08"/>
 </segment>
 <segment>
@@
 </segment>
 <segment>
-<wire x1="-2.54" y1="132.08" x2="12.7" y2="132.08" width="0.1524" layer="91"/>
+<wire x1="-2.54" y1="132.08" x2="7.62" y2="132.08" width="0.1524" layer="91"/>
 <pinref part="J.C6" gate="G$1" pin="2"/>
 <pinref part="I.J3" gate="G$1" pin="VBAT"/>
 <pinref part="J.C5" gate="G$1" pin="2"/>
+<wire x1="7.62" y1="132.08" x2="12.7" y2="132.08" width="0.1524" layer="91"/>
 <wire x1="25.4" y1="137.16" x2="12.7" y2="137.16" width="0.1524" layer="91"/>
 <wire x1="12.7" y1="137.16" x2="10.16" y2="137.16" width="0.1524" layer="91"/>
@@
 <wire x1="25.4" y1="132.08" x2="12.7" y2="132.08" width="0.1524" layer="91"/>
 <junction x="12.7" y="132.08"/>
-<wire x1="12.7" y1="121.92" x2="12.7" y2="129.54" width="0.1524" layer="91"/>
 <wire x1="12.7" y1="129.54" x2="12.7" y2="132.08" width="0.1524" layer="91"/>
 <wire x1="12.7" y1="137.16" x2="12.7" y2="132.08" width="0.1524" layer="91"/>
@@
 <pinref part="I.J3" gate="G$1" pin="BS1"/>
 <wire x1="25.4" y1="129.54" x2="12.7" y2="129.54" width="0.1524" layer="91"/>
-<junction x="12.7" y="129.54"/>
-<pinref part="I.J3" gate="G$1" pin="RES#"/>
-<wire x1="25.4" y1="121.92" x2="12.7" y2="121.92" width="0.1524" layer="91"/>
+<pinref part="J.R3" gate="G$1" pin="1"/>
+<junction x="7.62" y="132.08"/>
 </segment>
 </net>
@@
 </segment>
 </net>
+<net name="N$2" class="0">
+<segment>
+<pinref part="I.J3" gate="G$1" pin="RES#"/>
+<wire x1="25.4" y1="121.92" x2="7.62" y2="121.92" width="0.1524" layer="91"/>
+<pinref part="J.R3" gate="G$1" pin="2"/>
+<pinref part="J.C7" gate="G$1" pin="2"/>
+<wire x1="-2.54" y1="121.92" x2="7.62" y2="121.92" width="0.1524" layer="91"/>
+<junction x="7.62" y="121.92"/>
+</segment>
+</net>
