File: pcb/eagle/projects/size_M/D_ext_power/obsolete/M_D_ext_power_8_0_2.brd (EAGLE design)
At the start: 32 parts, among them U1 LM66100DCKR

Commit message: version 8 main changes * ideal diode separated 3v3 DC-DC to protect it from back current * smaller package of ina 219 * usage of tssop attiny v2 in adapter * and change of PA5 to PB2 with ^ and ~ (originally used for shield power switch - now PB3) * step motor shield * out signal for BT module
Parts:
- removed D.C6: 100n, rcl:C0603
- removed U1: LM66100DCKR, LM66100DCKR:SOT65P210X110-6N
- added D.D2: (no value), hugo:SHOTKY_2.8
- D.C4: device rcl:C0603 -> rcl:C0805
- D.D3: value SHOTKY_2.8 -> (none)
- D.U3: value (none) -> INA219AIDR; device hugo:SOT23-8 -> SamacSys_Parts:SOIC127P600X175-8N
- moved D.R4 4.78 mm to (6.17, 6.22)
- moved D.R7 4.22 mm to (2.91, 16.2), turned to 270 degrees
- moved D.C4 2.99 mm to (10.9, 17.1), turned to 180 degrees
- moved D.R3 2.98 mm to (8.45, 9.10), flipped to the bottom, turned to 180 degrees
- moved D.U3 2.38 mm to (6.58, 9.75), flipped to the top, turned to 0 degrees
- moved D.R6 1.75 mm to (4.60, 9.10), flipped to the bottom, turned to 0 degrees
- moved D.U1 0.69 mm to (5.28, 13.8)
- moved D.C5 0.46 mm to (9.25, 6.22), turned to 0 degrees
- moved D.L1 0.32 mm to (15.5, 16.1)
- moved D.C1 0.31 mm to (8.45, 7.20)
- moved D.U2 0.31 mm to (15.2, 12.6)
- moved D.R2 0.28 mm to (15.7, 3.00)
- moved D.LIPOL 0.25 mm to (5.65, 19.4)
- moved D.C3 0.24 mm to (17.7, 13.0)
- moved D.F2 0.17 mm to (17.2, 10.5)
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Connections:
- removed net VCC1: D.C4.2, D.L1.2, D.U2.BP, U1.1
- net GND: now also D.U3.6; no longer D.C6.1, D.U3.3, U1.2
- net IN+: now also D.LIPOL.3, D.R10.2, D.R5.1, D.U3.7; no longer D.C2.2, D.C3.2, D.F2.1, D.ON/OFF/RESET.P$2, D.ON/OFF/RESET.P$3, D.ON/OFF/RESET.P$4, D.ON/OFF/RESET.P$6, D.R10.1, D.U1.5, D.U1.8, D.U2.VIN, D.U3.1
- net IN-: now also D.C2.2, D.C3.2, D.D2.K, D.F2.1, D.ON/OFF/RESET.P$2, D.ON/OFF/RESET.P$3, D.ON/OFF/RESET.P$4, D.ON/OFF/RESET.P$6, D.R10.1, D.U1.5, D.U1.8, D.U2.VIN, D.U3.8; no longer D.LIPOL.3, D.R10.2, D.R5.1, D.U3.2
- net PA1: now also D.U3.2; no longer D.U3.7
- net PA2: now also D.U3.1; no longer D.U3.8
- net SCL: now also D.U3.4; no longer D.U3.5
- net SDA: now also D.U3.3; no longer D.U3.6
- net VCC: now also D.C4.2, D.D2.A, D.L1.2, D.U2.BP, D.U3.5; no longer D.C6.2, D.U3.4, U1.3, U1.6
Routing:
- net IN+: track 49.4 -> 17.2 mm, vias 7 -> 0
- net IN-: track 20.8 -> 51.2 mm, vias 1 -> 5
- net VCC1: track 15.4 -> 0.00 mm, vias 1 -> 0
- net VCC: track 20.2 -> 33.7 mm
- net GND: track 122.0 -> 111.3 mm, vias 14 -> 8
- net N$8: track 26.4 -> 23.2 mm
- net 5V: track 29.8 -> 27.1 mm, vias 1 -> 0
- net PA2: track 6.59 -> 4.18 mm
- net CHRG: track 7.93 -> 9.89 mm
- net PA1: track 4.84 -> 3.08 mm
- net PA3: track 10.0 -> 8.94 mm
- net N$7: track 4.65 -> 3.74 mm
- net N$3: track 7.58 -> 6.85 mm
- net SDA: track 3.10 -> 2.53 mm
- net SCL: track 2.45 -> 2.95 mm
