File: pcb/eagle/projects/size_M/H_ext_rgb/M_H_ext_rgb.brd (EAGLE design)
At the start: 6 parts

Commit message: PCB M.1
Parts:
- moved H.R1 0.43 mm to (5.30, 16.8)
- moved H.R2 0.41 mm to (5.30, 14.7)
- moved H.R3 0.36 mm to (5.30, 12.6)

Commit message: closed PCB version M.2
Other:
- board text added: "RGB M.2"
- board text removed: "RGB M.1"
Changed lines of the file:
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@@
 <hole x="2" y="2" drill="1.6"/>
 <circle x="2" y="2" radius="1.9" width="0.1" layer="52"/>
-<text x="6.0898" y="0.904" size="1.6764" layer="21">RGB M.1</text>
+<text x="6.0898" y="0.904" size="1.6764" layer="21">RGB M.2</text>
 <hole x="19" y="19" drill="1.6"/>
 <circle x="19" y="19" radius="1.9" width="0.1" layer="52"/>

Commit message: PCB v7 * 14 pin attiny is main adapter chip now. * changed adapter pin meaning (a1-a5, swapped RX-TX, VUSB replaced by A5, top most pin changed from GND to A4) * changed usb chip of main board
Parts:
- moved H.R1 11.3 mm to (16.4, 14.5), turned to 180 degrees
- moved H.R2 4.39 mm to (6.44, 18.9)
- moved H.R3 4.39 mm to (6.44, 16.9)
Connections:
- net GND: no longer H.J2.6
- net N$4: now also JP1.1; no longer H.J2.5
- net N$5: now also H.J2.6; no longer H.J2.4
- net N$6: now also H.J2.5; no longer H.J2.3
Routing:
- net GND: track 33.0 -> 11.5 mm, vias 0 -> 3
- net N$1: track 8.82 -> 4.90 mm
- net N$2: track 2.86 -> 5.22 mm
- net N$3: track 6.14 -> 8.03 mm
- net N$5: track 3.21 -> 4.38 mm
- net N$4: track 3.32 -> 2.43 mm
- net N$6: track 3.57 -> 4.20 mm
- added copper zone on layer 16, net GND
- removed copper zone on layer 16, net VDD
Other:
- board text added: "RGB M.7"
- board text removed: "RGB M.2"
Changed lines of the file:
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@@
 <setting verticaltext="up"/>
 </settings>
-<grid distance="1" unitdist="mm" unit="mm" style="lines" multiple="1" display="yes" altdistance="0.1" altunitdist="mm" altunit="mm"/>
+<grid distance="1" unitdist="mil" unit="mm" style="lines" multiple="1" display="yes" altdistance="0.1" altunitdist="mm" altunit="mm"/>
 <layers>
 <layer number="1" name="Top" color="4" fill="1" visible="yes" active="yes"/>
@@
 <hole x="2" y="2" drill="1.6"/>
 <circle x="2" y="2" radius="1.9" width="0.1" layer="52"/>
-<text x="6.0898" y="0.904" size="1.6764" layer="21">RGB M.2</text>
+<text x="6.0898" y="0.904" size="1.6764" layer="21">RGB M.7</text>
 <hole x="19" y="19" drill="1.6"/>
 <circle x="19" y="19" radius="1.9" width="0.1" layer="52"/>
@@
 <param name="mtCopper" value="0.035mm 0.035mm 0.035mm 0.035mm 0.035mm 0.035mm 0.035mm 0.035mm 0.035mm 0.035mm 0.035mm 0.035mm 0.035mm 0.035mm 0.035mm 0.035mm"/>
 <param name="mtIsolate" value="1.5mm 0.15mm 0.2mm 0.15mm 0.2mm 0.15mm 0.2mm 0.15mm 0.2mm 0.15mm 0.2mm 0.15mm 0.2mm 0.15mm 0.2mm"/>
-<param name="mdWireWire" value="14mil"/>
-<param name="mdWirePad" value="13mil"/>
-<param name="mdWireVia" value="14mil"/>
+<param name="mdWireWire" value="10mil"/>
+<param name="mdWirePad" value="10mil"/>
+<param name="mdWireVia" value="10mil"/>
 <param name="mdPadPad" value="10mil"/>
-<param name="mdPadVia" value="14mil"/>
-<param name="mdViaVia" value="14mil"/>
-<param name="mdSmdPad" value="14mil"/>
-<param name="mdSmdVia" value="14mil"/>
-<param name="mdSmdSmd" value="14mil"/>
+<param name="mdPadVia" value="10mil"/>
+<param name="mdViaVia" value="10mil"/>
+<param name="mdSmdPad" value="10mil"/>
+<param name="mdSmdVia" value="10mil"/>
+<param name="mdSmdSmd" value="10mil"/>
 <param name="mdViaViaSameLayer" value="6mil"/>
 <param name="mnLayersViaInSmd" value="2"/>
-<param name="mdCopperDimension" value="15mil"/>
+<param name="mdCopperDimension" value="10mil"/>
 <param name="mdDrill" value="15mil"/>
 <param name="mdSmdStop" value="0mil"/>
@@
 </element>
 <element name="H.D1" library="hugo" package="RGB_WW-FCE50TC-Q1" value="RGB_WW-FCE50TC-Q1" x="10.554" y="10.454" smashed="yes" rot="R180"/>
-<element name="H.R1" library="resistor" package="R0603" value="82" x="5.3" y="16.7842" smashed="yes">
-<attribute name="NAME" x="3.9538" y="17.543" size="0.889" layer="25"/>
+<element name="H.R1" library="resistor" package="R0603" value="82" x="16.3952" y="14.4952" smashed="yes" rot="R180">
+<attribute name="NAME" x="17.7414" y="13.7364" size="0.889" layer="25" rot="R180"/>
 </element>
-<element name="H.R2" library="resistor" package="R0603" value="82" x="5.3" y="14.7046" smashed="yes">
-<attribute name="NAME" x="7.7344" y="13.1778" size="0.889" layer="25" rot="R90"/>
+<element name="H.R2" library="resistor" package="R0603" value="82" x="6.443" y="18.9464" smashed="yes">
+<attribute name="NAME" x="8.124" y="18.5054" size="0.889" layer="25"/>
 </element>
-<element name="H.R3" library="resistor" package="R0603" value="82" x="5.3" y="12.6144" smashed="yes">
-<attribute name="NAME" x="3.876" y="11.0114" size="0.889" layer="25"/>
+<element name="H.R3" library="resistor" package="R0603" value="82" x="6.443" y="16.8562" smashed="yes">
+<attribute name="NAME" x="8.1432" y="16.4216" size="0.889" layer="25"/>
 </element>
 <element name="JP1" library="pinhead2" package="1X04" package3d_urn="urn:adsk.eagle:package:22407/2" value="" x="19.6" y="10.5" smashed="yes" rot="R270">
@@
 <wire x1="8.832" y1="8.34" x2="10.582" y2="8.34" width="0.3556" layer="1"/>
 <wire x1="10.582" y1="8.34" x2="12.332" y2="8.34" width="0.3556" layer="1"/>
-<polygon width="0.3048" layer="1" isolate="0.3048">
+<polygon width="0.254" layer="1" isolate="0.254">
 <vertex x="0.5" y="20.5"/>
 <vertex x="0.5" y="0.5"/>
@@
 <wire x1="12.332" y1="8.34" x2="13.8814" y2="8.34" width="0.3556" layer="1"/>
 <wire x1="13.8814" y1="8.34" x2="13.9068" y2="8.34" width="0.3556" layer="1"/>
-<wire x1="14.6444" y1="9.0776" x2="13.9068" y2="8.34" width="0.3556" layer="1"/>
-<contactref element="H.J2" pad="6"/>
-<wire x1="14.3422" y1="14.4878" x2="14.3276" y2="14.4878" width="0.3556" layer="1"/>
-<wire x1="14.3276" y1="14.4878" x2="14.6444" y2="14.171" width="0.3556" layer="1"/>
-<wire x1="14.6444" y1="14.171" x2="14.6444" y2="9.0776" width="0.3556" layer="1"/>
 <wire x1="19.6" y1="6.69" x2="15.5314" y2="6.69" width="0.3556" layer="1"/>
 <wire x1="15.5314" y1="6.69" x2="13.8814" y2="8.34" width="0.3556" layer="1"/>
 <contactref element="JP1" pad="4"/>
-<wire x1="1.4" y1="19.39" x2="9.4254" y2="19.39" width="0.3556" layer="1"/>
-<wire x1="9.4254" y1="19.39" x2="14.3276" y2="14.4878" width="0.3556" layer="1"/>
-</signal>
-<signal name="N$3">
-<contactref element="H.R2" pad="2"/>
-<contactref element="H.D1" pad="2"/>
-<wire x1="10.582" y1="12.74" x2="10.582" y2="14.2592" width="0.3556" layer="1"/>
-<wire x1="10.582" y1="14.2592" x2="10.16" y2="14.6812" width="0.3556" layer="1"/>
-<wire x1="10.16" y1="14.6812" x2="6.173921875" y2="14.6812" width="0.3556" layer="1"/>
-<wire x1="6.173921875" y1="14.6812" x2="6.15" y2="14.7046" width="0.3556" layer="1"/>
-</signal>
-<signal name="N$1">
-<contactref element="H.R1" pad="2"/>
-<contactref element="H.D1" pad="1"/>
-<wire x1="12.332" y1="12.74" x2="12.3812" y2="12.7892" width="0.3556" layer="1"/>
-<wire x1="10.1652" y1="16.454" x2="6.51486875" y2="16.454" width="0.3556" layer="1"/>
-<wire x1="6.15" y1="16.7842" x2="6.51486875" y2="16.454" width="0.3556" layer="1"/>
-<wire x1="12.332" y1="14.2872" x2="12.332" y2="12.74" width="0.3556" layer="1"/>
-<wire x1="10.1652" y1="16.454" x2="12.332" y2="14.2872" width="0.3556" layer="1"/>
-</signal>
-<signal name="N$2">
-<contactref element="H.R3" pad="2"/>
-<contactref element="H.D1" pad="3"/>
-<wire x1="8.832" y1="12.74" x2="8.6782" y2="12.8938" width="0.3556" layer="1"/>
-<wire x1="8.6782" y1="12.8938" x2="6.4294" y2="12.8938" width="0.3556" layer="1"/>
-<wire x1="6.4294" y1="12.8938" x2="6.15" y2="12.6144" width="0.3556" layer="1"/>
-</signal>
-<signal name="VDD">
-<polygon width="0.3048" layer="16" isolate="0.3048">
+<via x="19.558" y="16.5354" extent="1-16" drill="0.35"/>
+<polygon width="0.254" layer="16" isolate="0.254">
 <vertex x="0.5" y="20.5"/>
 <vertex x="0.5" y="0.5"/>
@@
 <vertex x="20.5" y="20.5"/>
 </polygon>
+<via x="1.4224" y="4.4196" extent="1-16" drill="0.35"/>
+<via x="3.3274" y="20.1168" extent="1-16" drill="0.35"/>
+</signal>
+<signal name="N$3">
+<contactref element="H.R2" pad="2"/>
+<contactref element="H.D1" pad="2"/>
+<wire x1="10.582" y1="12.74" x2="10.582" y2="16.471671875" width="0.3556" layer="1"/>
+<wire x1="10.582" y1="16.471671875" x2="8.05924375" y2="18.9464" width="0.3556" layer="1"/>
+<wire x1="7.293" y1="18.9464" x2="8.05924375" y2="18.9464" width="0.3556" layer="1"/>
+</signal>
+<signal name="N$1">
+<contactref element="H.R1" pad="2"/>
+<contactref element="H.D1" pad="1"/>
+<wire x1="12.332" y1="12.74" x2="12.3812" y2="12.7892" width="0.3556" layer="1"/>
+<wire x1="15.5452" y1="14.4952" x2="15.5198" y2="14.4698" width="0.3556" layer="1"/>
+<wire x1="15.5198" y1="14.4698" x2="12.5394" y2="14.4698" width="0.3556" layer="1"/>
+<wire x1="12.332" y1="14.2624" x2="12.332" y2="12.74" width="0.3556" layer="1"/>
+<wire x1="12.5394" y1="14.4698" x2="12.332" y2="14.2624" width="0.3556" layer="1"/>
+</signal>
+<signal name="N$2">
+<contactref element="H.R3" pad="2"/>
+<contactref element="H.D1" pad="3"/>
+<wire x1="8.832" y1="16.1182" x2="8.094" y2="16.8562" width="0.3556" layer="1"/>
+<wire x1="7.293" y1="16.8562" x2="8.094" y2="16.8562" width="0.3556" layer="1"/>
+<wire x1="8.832" y1="12.74" x2="8.832" y2="16.1182" width="0.3556" layer="1"/>
+</signal>
+<signal name="VDD">
 <contactref element="JP1" pad="3"/>
 </signal>
 <signal name="N$4">
+<contactref element="JP1" pad="1"/>
 <contactref element="H.R1" pad="1"/>
-<contactref element="H.J2" pad="5"/>
-<wire x1="4.45" y1="16.7842" x2="4.1452" y2="16.4794" width="0.3556" layer="1"/>
-<wire x1="4.1452" y1="16.4794" x2="1.804815625" y2="16.4794" width="0.3556" layer="1"/>
-<wire x1="1.804815625" y1="16.4794" x2="1.4" y2="16.85" width="0.3556" layer="1"/>
+<wire x1="19.6" y1="14.31" x2="19.4148" y2="14.4952" width="0.3556" layer="1"/>
+<wire x1="19.4148" y1="14.4952" x2="17.2452" y2="14.4952" width="0.3556" layer="1"/>
 </signal>
 <signal name="N$5">
-<contactref element="H.J2" pad="4"/>
 <contactref element="H.R2" pad="1"/>
-<wire x1="1.4" y1="14.31" x2="1.7946" y2="14.7046" width="0.3556" layer="1"/>
-<wire x1="4.45" y1="14.7046" x2="1.7946" y2="14.7046" width="0.3556" layer="1"/>
+<contactref element="H.J2" pad="6"/>
+<wire x1="1.8436" y1="18.9464" x2="1.4" y2="19.39" width="0.3556" layer="1"/>
+<wire x1="5.593" y1="18.9464" x2="1.8436" y2="18.9464" width="0.3556" layer="1"/>
 </signal>
 <signal name="N$6">
 <contactref element="H.R3" pad="1"/>
-<contactref element="H.J2" pad="3"/>
-<wire x1="4.45" y1="12.6144" x2="4.1706" y2="12.8938" width="0.3556" layer="1"/>
-<wire x1="4.1706" y1="12.8938" x2="2.769178125" y2="12.8938" width="0.3556" layer="1"/>
-<wire x1="1.4" y1="11.77" x2="2.769178125" y2="12.8938" width="0.3556" layer="1"/>
+<wire x1="5.593" y1="16.8562" x2="2.184978125" y2="16.8562" width="0.3556" layer="1"/>
+<contactref element="H.J2" pad="5"/>
+<wire x1="1.4" y1="16.85" x2="2.178778125" y2="16.85" width="0.3556" layer="1"/>
+<wire x1="2.178778125" y1="16.85" x2="2.184978125" y2="16.8562" width="0.3556" layer="1"/>
 </signal>
 </signals>

Commit message: PCB v9
Parts:
- removed JP1: (no value), pinhead2:1X04
- added H.J1: (no value), pinhead2:1X06
- moved H.R1 4.76 mm to (16.2, 9.74), turned to 90 degrees
Connections:
- net GND: now also H.J1.4; no longer JP1.4
- net N$4: now also H.J1.6; no longer JP1.1
- net VDD: now also H.J1.3; no longer JP1.3
Routing:
- net N$4: track 2.43 -> 9.24 mm, vias 0 -> 1
- net GND: vias 3 -> 4
Other:
- board text added: "RGB M.9"
- board text removed: "RGB M.7"
Changed lines of the file:
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@@
 <setting verticaltext="up"/>
 </settings>
-<grid distance="1" unitdist="mil" unit="mm" style="lines" multiple="1" display="yes" altdistance="0.1" altunitdist="mm" altunit="mm"/>
+<grid distance="0.5" unitdist="mm" unit="mm" style="lines" multiple="1" display="yes" altdistance="0.1" altunitdist="mm" altunit="mm"/>
 <layers>
 <layer number="1" name="Top" color="4" fill="1" visible="yes" active="yes"/>
@@
 <hole x="2" y="2" drill="1.6"/>
 <circle x="2" y="2" radius="1.9" width="0.1" layer="52"/>
-<text x="6.0898" y="0.904" size="1.6764" layer="21">RGB M.7</text>
+<text x="6.0898" y="0.904" size="1.6764" layer="21">RGB M.9</text>
 <hole x="19" y="19" drill="1.6"/>
 <circle x="19" y="19" radius="1.9" width="0.1" layer="52"/>
@@
 </element>
 <element name="H.D1" library="hugo" package="RGB_WW-FCE50TC-Q1" value="RGB_WW-FCE50TC-Q1" x="10.554" y="10.454" smashed="yes" rot="R180"/>
-<element name="H.R1" library="resistor" package="R0603" value="82" x="16.3952" y="14.4952" smashed="yes" rot="R180">
-<attribute name="NAME" x="17.7414" y="13.7364" size="0.889" layer="25" rot="R180"/>
+<element name="H.R1" library="resistor" package="R0603" value="82" x="16.1716" y="9.7414" smashed="yes" rot="R90">
+<attribute name="NAME" x="15.4128" y="8.3952" size="0.889" layer="25" rot="R90"/>
 </element>
 <element name="H.R2" library="resistor" package="R0603" value="82" x="6.443" y="18.9464" smashed="yes">
@@
 <attribute name="NAME" x="8.1432" y="16.4216" size="0.889" layer="25"/>
 </element>
-<element name="JP1" library="pinhead2" package="1X04" package3d_urn="urn:adsk.eagle:package:22407/2" value="" x="19.6" y="10.5" smashed="yes" rot="R270">
-<attribute name="POPULARITY" value="91" x="19.6" y="10.5" size="1.778" layer="27" rot="R270" display="off"/>
+<element name="H.J1" library="pinhead2" package="1X06" package3d_urn="urn:adsk.eagle:package:22472/2" value="" x="19.6" y="7.96" smashed="yes" rot="R270">
+<attribute name="POPULARITY" value="79" x="19.6" y="7.96" size="1.778" layer="27" rot="R270" display="off"/>
 <attribute name="VALUE" x="16.425" y="15.58" size="1.27" layer="27" rot="R270"/>
 </element>
@@
 <vertex x="20.5" y="20.5"/>
 </polygon>
-<wire x1="12.332" y1="8.34" x2="13.8814" y2="8.34" width="0.3556" layer="1"/>
-<wire x1="13.8814" y1="8.34" x2="13.9068" y2="8.34" width="0.3556" layer="1"/>
-<wire x1="19.6" y1="6.69" x2="15.5314" y2="6.69" width="0.3556" layer="1"/>
-<wire x1="15.5314" y1="6.69" x2="13.8814" y2="8.34" width="0.3556" layer="1"/>
-<contactref element="JP1" pad="4"/>
-<via x="19.558" y="16.5354" extent="1-16" drill="0.35"/>
+<wire x1="15.252" y1="6.69" x2="13.602" y2="8.34" width="0.3556" layer="1"/>
+<wire x1="13.602" y1="8.34" x2="12.332" y2="8.34" width="0.3556" layer="1"/>
+<wire x1="19.6" y1="6.69" x2="15.252" y2="6.69" width="0.3556" layer="1"/>
+<via x="19.558" y="16.5354" extent="1-16" drill="0.3"/>
 <polygon width="0.254" layer="16" isolate="0.254">
 <vertex x="0.5" y="20.5"/>
@@
 <vertex x="20.5" y="20.5"/>
 </polygon>
-<via x="1.4224" y="4.4196" extent="1-16" drill="0.35"/>
-<via x="3.3274" y="20.1168" extent="1-16" drill="0.35"/>
+<via x="1.4224" y="4.4196" extent="1-16" drill="0.3"/>
+<via x="3.3274" y="20.1168" extent="1-16" drill="0.3"/>
+<contactref element="H.J1" pad="4"/>
+<via x="17.2974" y="1.2954" extent="1-16" drill="0.3"/>
+<wire x1="19.6" y1="6.69" x2="19.558" y2="16.5354" width="0" layer="19" extent="1-1"/>
+<wire x1="17.2974" y1="1.2954" x2="19.6" y2="6.69" width="0" layer="19" extent="1-1"/>
+<wire x1="1.4224" y1="4.4196" x2="8.832" y2="8.34" width="0" layer="19" extent="1-1"/>
+<wire x1="3.3274" y1="20.1168" x2="8.832" y2="8.34" width="0" layer="19" extent="1-1"/>
 </signal>
 <signal name="N$3">
 <contactref element="H.R2" pad="2"/>
 <contactref element="H.D1" pad="2"/>
-<wire x1="10.582" y1="12.74" x2="10.582" y2="16.471671875" width="0.3556" layer="1"/>
-<wire x1="10.582" y1="16.471671875" x2="8.05924375" y2="18.9464" width="0.3556" layer="1"/>
-<wire x1="7.293" y1="18.9464" x2="8.05924375" y2="18.9464" width="0.3556" layer="1"/>
+<wire x1="9.6168" y1="16.675128125" x2="9.6168" y2="14.7974" width="0.3556" layer="1"/>
+<wire x1="10.582" y1="12.74" x2="10.582" y2="13.8322" width="0.3556" layer="1"/>
+<wire x1="10.582" y1="13.8322" x2="9.6168" y2="14.7974" width="0.3556" layer="1"/>
+<wire x1="9.6168" y1="16.675128125" x2="7.301446875" y2="18.9464" width="0.3556" layer="1"/>
+<wire x1="7.293" y1="18.9464" x2="7.301446875" y2="18.9464" width="0.3556" layer="1"/>
 </signal>
 <signal name="N$1">
@@
 <contactref element="H.D1" pad="1"/>
 <wire x1="12.332" y1="12.74" x2="12.3812" y2="12.7892" width="0.3556" layer="1"/>
-<wire x1="15.5452" y1="14.4952" x2="15.5198" y2="14.4698" width="0.3556" layer="1"/>
-<wire x1="15.5198" y1="14.4698" x2="12.5394" y2="14.4698" width="0.3556" layer="1"/>
-<wire x1="12.332" y1="14.2624" x2="12.332" y2="12.74" width="0.3556" layer="1"/>
-<wire x1="12.5394" y1="14.4698" x2="12.332" y2="14.2624" width="0.3556" layer="1"/>
+<wire x1="16.1716" y1="10.5914" x2="15.4858" y2="11.2772" width="0.3556" layer="1"/>
+<wire x1="15.4858" y1="11.2772" x2="13.0328" y2="11.2772" width="0.3556" layer="1"/>
+<wire x1="13.0328" y1="11.2772" x2="12.332" y2="11.978" width="0.3556" layer="1"/>
+<wire x1="12.332" y1="11.978" x2="12.332" y2="12.74" width="0.3556" layer="1"/>
 </signal>
 <signal name="N$2">
 <contactref element="H.R3" pad="2"/>
 <contactref element="H.D1" pad="3"/>
-<wire x1="8.832" y1="16.1182" x2="8.094" y2="16.8562" width="0.3556" layer="1"/>
-<wire x1="7.293" y1="16.8562" x2="8.094" y2="16.8562" width="0.3556" layer="1"/>
-<wire x1="8.832" y1="12.74" x2="8.832" y2="16.1182" width="0.3556" layer="1"/>
+<wire x1="8.832" y1="16.2198" x2="8.1956" y2="16.8562" width="0.3556" layer="1"/>
+<wire x1="7.293" y1="16.8562" x2="8.1956" y2="16.8562" width="0.3556" layer="1"/>
+<wire x1="8.832" y1="12.74" x2="8.832" y2="16.2198" width="0.3556" layer="1"/>
 </signal>
 <signal name="VDD">
-<contactref element="JP1" pad="3"/>
+<contactref element="H.J1" pad="3"/>
 </signal>
 <signal name="N$4">
-<contactref element="JP1" pad="1"/>
 <contactref element="H.R1" pad="1"/>
-<wire x1="19.6" y1="14.31" x2="19.4148" y2="14.4952" width="0.3556" layer="1"/>
-<wire x1="19.4148" y1="14.4952" x2="17.2452" y2="14.4952" width="0.3556" layer="1"/>
+<contactref element="H.J1" pad="6"/>
+<wire x1="16.1716" y1="8.8914" x2="16.1716" y2="7.7552" width="0.3556" layer="1"/>
+<wire x1="16.1716" y1="7.7552" x2="16.1798" y2="7.747" width="0.3556" layer="1"/>
+<via x="16.1798" y="7.747" extent="1-16" drill="0.3"/>
+<wire x1="16.1798" y1="7.747" x2="16.1798" y2="4.1158" width="0.3556" layer="16"/>
+<wire x1="18.6856" y1="1.61" x2="16.1798" y2="4.1158" width="0.3556" layer="16"/>
+<wire x1="18.6856" y1="1.61" x2="19.6" y2="1.61" width="0.3556" layer="16"/>
 </signal>
 <signal name="N$5">
