File: pcb/eagle/projects/size_M/B_adapter/M_B_adapter-tssop.brd (EAGLE design)
At the start: 16 parts

Commit message: formal changes - resistors renamed
Parts:
- B.R3: value 330 -> 390
- renumbered B.R7 to B.R5
Changed lines of the file:
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@@
 <attribute name="VALUE" x="9.525" y="7.9248" size="1.27" layer="27" rot="R270"/>
 </element>
-<element name="B.R7" library="hugo" package="FUSE" value="alt fuse or 0R" x="16.9418" y="10.2514" smashed="yes" rot="R90">
+<element name="B.R5" library="hugo" package="FUSE" value="alt fuse or 0R" x="16.9418" y="10.2514" smashed="yes" rot="R90">
 <attribute name="NAME" x="17.0434" y="11.9786" size="0.8128" layer="25" rot="R90"/>
 <attribute name="VALUE" x="18.8468" y="9.6164" size="1.27" layer="27" rot="R90"/>
 </element>
-<element name="B.R3" library="rcl" library_urn="urn:adsk.eagle:library:334" package="R0603" package3d_urn="urn:adsk.eagle:package:23555/3" value="330" x="14.7" y="19.3328" smashed="yes" rot="R180">
+<element name="B.R3" library="rcl" library_urn="urn:adsk.eagle:library:334" package="R0603" package3d_urn="urn:adsk.eagle:package:23555/3" value="390" x="14.7" y="19.3328" smashed="yes" rot="R180">
 <attribute name="NAME" x="13.4006" y="20.0594" size="0.8128" layer="25"/>
 <attribute name="POPULARITY" value="70" x="14.7" y="13.8972" size="1.778" layer="27" rot="R180" display="off"/>
@@
 <wire x1="13.04" y1="15.07081875" x2="13.04" y2="15.45608125" width="0.6096" layer="16"/>
 <wire x1="11.77" y1="12.3317875" x2="13.04" y2="13.6017875" width="0.6096" layer="16"/>
-<contactref element="B.R7" pad="2"/>
+<contactref element="B.R5" pad="2"/>
 <wire x1="16.5862" y1="10.8458" x2="16.9418" y2="11.2014" width="0.508" layer="1"/>
 <contactref element="B.R1" pad="2"/>
@@
 <contactref element="B.T1" pad="D"/>
 <contactref element="B.C1" pad="1"/>
-<contactref element="B.R7" pad="1"/>
+<contactref element="B.R5" pad="1"/>
 <wire x1="16.9418" y1="7.5556" x2="16.9672" y2="7.5302" width="0.508" layer="1"/>
 <wire x1="13.9446" y1="9.4312" x2="14.1506" y2="9.2252" width="0.6096" layer="1"/>
